File: 3000.kicad_pcb (KiCad board)
At the start: 2 copper layers, 449.1 x 144.3 mm, 460 parts, among them J1 CONN_01X04, Q1 SI2305, SW1 SWITCH, U1 ATMEGA32U4, U1_2 ATMEGA32U4, X1 16MHz

Commit message: draw
Parts:
- removed the REF** at (456.7, 126.2)
- removed the REF** at (447.7, 127.3)
- added LED7: 3mm, Keyboard:LED_D3.0mm, F.Cu at (114.5, 148.3)
- added LED8: 3mm, Keyboard:LED_D3.0mm, F.Cu at (112.0, 148.3)
- added R10: 330R, Keyboard:R_0805, B.Cu at (110.7, 143.2)
- added R9: 330R, Keyboard:R_0805, B.Cu at (115.8, 143.2)
- added REF**: Hole, Keyboard:Hole, F.Cu at (454.9, 128.7)
- added REF**: Hole, Keyboard:Hole, F.Cu at (447.5, 128.7)
- added RGB: Pin_Header_Straight_1x03_Pitch2.54mm, Pin_Headers:Pin_Header_Straight_1x03_Pitch2.54mm, B.Cu at (115.8, 138.2)
- RGBLED1, RGBLED2, RGBLED3, RGBLED4: footprint 3000:SK6812mini_BackSMD -> Keyboard:SK6812mini_BackSMD
- moved RGBLED4 46.0 mm to (88.4, 137.4), turned to 225 degrees
- moved RGBLED2 45.6 mm to (100.0, 149.0)
- moved RGBLED3 43.4 mm to (88.4, 149.0), turned to 270 degrees
- moved C11 42.9 mm to (94.2, 151.6)
- moved RGBLED1 42.4 mm to (100.0, 137.4), turned to 90 degrees
- moved C10 30.8 mm to (102.8, 143.2)
- moved KBD1 21.6 mm to (106.8, 140.7)
- moved KBR1 21.6 mm to (106.8, 148.3)
- moved C12 21.0 mm to (85.6, 143.2), turned to 180 degrees
- moved C9 20.6 mm to (94.2, 134.9), turned to 180 degrees
Connections:
- RGBLED1 pad 3: /RGBIN -> /LED3
Routing:
- net GND: track 3662.9 -> 4161.3 mm
- net /LED3: track 58.2 -> 490.2 mm
- net VCC: track 262.7 -> 687.6 mm
- net /LED+: track 7538.2 -> 7493.8 mm
- net /ROW5: track 745.5 -> 709.0 mm
- net /ROW4: track 738.0 -> 701.5 mm
- net /ROW3: track 704.9 -> 668.4 mm
- net /ROW6: track 909.3 -> 874.4 mm
- net Net-(KBR1-Pad1): track 6.75 -> 27.4 mm, vias 0 -> 1
- net Net-(KBD1-Pad1): track 4.22 -> 23.7 mm, vias 0 -> 1
- net /ROW1: track 610.6 -> 626.9 mm
- net Net-(RGBLED2-Pad1): track 0.00 -> 13.8 mm
- net Net-(RGBLED1-Pad1): track 0.00 -> 11.9 mm
- net Net-(RGBLED3-Pad1): track 0.00 -> 11.7 mm
- net /COL1: track 1019.1 -> 1008.7 mm
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- removed copper zone on F.Cu, net (none)
