File: 3000.sch (KiCad schematic (older format))
At the start: 389 parts, among them J1 CONN_01X04, Q1 SI2305, SW1 SWITCH, U1 ATMEGA32U4, U1_2 ATMEGA32U4, X1 16MHz

Commit message: draw
Parts:
- added LED7, LED8: 3mm, Keyboard:LED_D3.0mm, symbol LED
- added R10, R9: 330R, Keyboard:R_0805, symbol R
- RGBLED1, RGBLED2, RGBLED3, RGBLED4: footprint 3000:SK6812mini_BackSMD -> Keyboard:SK6812mini_BackSMD
- SW1: symbol SWITCH -> SWITCH-RESCUE-3000
Connections:
- net RGBIN is gone; now on net LED3: RGBLED1.3 (DIN)
- net GND: now also LED7.1 (K), LED8.1 (K)
- net LED+: now also R10.2, R9.2
- new net: LED7.2 (A), R9.1
- new net: LED8.2 (A), R10.1
Changed lines of the file:
@@
 LIBS:contrib
 LIBS:valves
-LIBS:3000
+LIBS:keyboard
 LIBS:3000-cache
 EELAYER 25 0
@@
 $EndComp
 $Comp
-L SWITCH SW1
+L SWITCH-RESCUE-3000 SW1
 U 1 1 58CF7BB0
 P 4150 12750
@@
 $EndComp
 $Comp
-L VCC #PWR08
+L VCC #PWR01
 U 1 1 595DA636
 P 3650 7700
-F 0 "#PWR08" H 3650 7550 50  0001 C CNN
+F 0 "#PWR01" H 3650 7550 50  0001 C CNN
 F 1 "VCC" H 3650 7850 50  0000 C CNN
 F 2 "" H 3650 7700 50  0001 C CNN
@@
 $EndComp
 $Comp
-L VCC #PWR09
+L VCC #PWR02
 U 1 1 5960435C
 P 9100 8950
-F 0 "#PWR09" H 9100 8800 50  0001 C CNN
+F 0 "#PWR02" H 9100 8800 50  0001 C CNN
 F 1 "VCC" H 9100 9100 50  0000 C CNN
 F 2 "" H 9100 8950 50  0001 C CNN
@@
 $EndComp
 $Comp
-L VCC #PWR010
+L VCC #PWR03
 U 1 1 59611212
 P 3800 12100
-F 0 "#PWR010" H 3800 11950 50  0001 C CNN
+F 0 "#PWR03" H 3800 11950 50  0001 C CNN
 F 1 "VCC" H 3800 12250 50  0000 C CNN
 F 2 "" H 3800 12100 50  0001 C CNN
@@
 $EndComp
 $Comp
-L VCC #PWR011
+L VCC #PWR04
 U 1 1 59613BCD
 P 5500 12100
-F 0 "#PWR011" H 5500 11950 50  0001 C CNN
+F 0 "#PWR04" H 5500 11950 50  0001 C CNN
 F 1 "VCC" H 5500 12250 50  0000 C CNN
 F 2 "" H 5500 12100 50  0001 C CNN
@@
 $EndComp
 $Comp
-L VCC #PWR012
+L VCC #PWR05
 U 1 1 59614E11
 P 7050 12100
-F 0 "#PWR012" H 7050 11950 50  0001 C CNN
+F 0 "#PWR05" H 7050 11950 50  0001 C CNN
 F 1 "VCC" H 7050 12250 50  0000 C CNN
 F 2 "" H 7050 12100 50  0001 C CNN
@@
 COL8
 $Comp
-L VCC #PWR013
+L VCC #PWR06
 U 1 1 59722202
 P 9800 10050
-F 0 "#PWR013" H 9800 9900 50  0001 C CNN
+F 0 "#PWR06" H 9800 9900 50  0001 C CNN
 F 1 "VCC" H 9800 10200 50  0000 C CNN
 F 2 "" H 9800 10050 50  0001 C CNN
@@
 $EndComp
 $Comp
-L VCC #PWR014
+L VCC #PWR07
 U 1 1 59A7212B
 P 3950 5900
-F 0 "#PWR014" H 3950 5750 50  0001 C CNN
+F 0 "#PWR07" H 3950 5750 50  0001 C CNN
 F 1 "VCC" H 3950 6050 50  0000 C CNN
 F 2 "" H 3950 5900 50  0001 C CNN
@@
 $EndComp
 $Comp
-L VCC #PWR015
+L VCC #PWR08
 U 1 1 59B329C2
 P 6100 6400
-F 0 "#PWR015" H 6100 6250 50  0001 C CNN
+F 0 "#PWR08" H 6100 6250 50  0001 C CNN
 F 1 "VCC" H 6100 6550 50  0000 C CNN
 F 2 "" H 6100 6400 50  0001 C CNN
@@
 NoConn ~ 5000 6650
 $Comp
-L VCC #PWR019
+L VCC #PWR09
 U 1 1 59BC5A75
 P 5000 5900
-F 0 "#PWR019" H 5000 5750 50  0001 C CNN
+F 0 "#PWR09" H 5000 5750 50  0001 C CNN
 F 1 "VCC" H 5000 6050 50  0000 C CNN
 F 2 "" H 5000 5900 50  0001 C CNN
@@
 F 0 "RGBLED4" H 9150 11700 60  0000 C CNN
 F 1 "SK6812_MINI" H 9150 11300 60  0000 C CNN
-F 2 "3000:SK6812mini_BackSMD" H 9200 11400 60  0000 C CNN
+F 2 "Keyboard:SK6812mini_BackSMD" H 9200 11400 60  0000 C CNN
 F 3 "" H 9200 11400 60  0000 C CNN
 	1    9150 11450
@@
 F 0 "RGBLED3" H 9150 12200 60  0000 C CNN
 F 1 "SK6812_MINI" H 9150 11800 60  0000 C CNN
-F 2 "3000:SK6812mini_BackSMD" H 9200 11900 60  0000 C CNN
+F 2 "Keyboard:SK6812mini_BackSMD" H 9200 11900 60  0000 C CNN
 F 3 "" H 9200 11900 60  0000 C CNN
 	1    9150 11950
@@
 F 0 "RGBLED2" H 9150 12700 60  0000 C CNN
 F 1 "SK6812_MINI" H 9150 12300 60  0000 C CNN
-F 2 "3000:SK6812mini_BackSMD" H 9200 12400 60  0000 C CNN
+F 2 "Keyboard:SK6812mini_BackSMD" H 9200 12400 60  0000 C CNN
 F 3 "" H 9200 12400 60  0000 C CNN
 	1    9150 12450
@@
 F 0 "RGBLED1" H 9150 13200 60  0000 C CNN
 F 1 "SK6812_MINI" H 9150 12800 60  0000 C CNN
-F 2 "3000:SK6812mini_BackSMD" H 9200 12900 60  0000 C CNN
+F 2 "Keyboard:SK6812mini_BackSMD" H 9200 12900 60  0000 C CNN
 F 3 "" H 9200 12900 60  0000 C CNN
 	1    9150 12950
@@
 	13300 5200 27700 5200
 Wire Wire Line
-	13600 3950 13600 3600
+	13600 3600 13600 4750
 Connection ~ 13600 3600
 Wire Wire Line
@@
 Connection ~ 9500 10750
 $Comp
-L VCC #PWR022
+L VCC #PWR010
 U 1 1 59EA085E
 P 9700 10750
-F 0 "#PWR022" H 9700 10600 50  0001 C CNN
+F 0 "#PWR010" H 9700 10600 50  0001 C CNN
 F 1 "VCC" H 9700 10900 50  0000 C CNN
 F 2 "" H 9700 10750 50  0001 C CNN
@@
 	1    0    0    -1
 $EndComp
-Text Label 9700 13000 2    60   ~ 0
-RGBIN
 $Comp
-L GND #PWR?
+L GND #PWR011
 U 1 1 59F7D83F
 P 9100 8450
-F 0 "#PWR?" H 9100 8200 50  0001 C CNN
+F 0 "#PWR011" H 9100 8200 50  0001 C CNN
 F 1 "GND" H 9100 8300 50  0000 C CNN
 F 2 "" H 9100 8450 50  0001 C CNN
@@
 $EndComp
 $Comp
-L GND #PWR?
+L GND #PWR012
 U 1 1 59F7E2FF
 P 3550 6850
-F 0 "#PWR?" H 3550 6600 50  0001 C CNN
+F 0 "#PWR012" H 3550 6600 50  0001 C CNN
 F 1 "GND" H 3550 6700 50  0000 C CNN
 F 2 "" H 3550 6850 50  0001 C CNN
@@
 $EndComp
 $Comp
-L GND #PWR?
+L GND #PWR013
 U 1 1 59F84460
 P 3650 6850
-F 0 "#PWR?" H 3650 6600 50  0001 C CNN
+F 0 "#PWR013" H 3650 6600 50  0001 C CNN
 F 1 "GND" H 3650 6700 50  0000 C CNN
 F 2 "" H 3650 6850 50  0001 C CNN
@@
 $EndComp
 $Comp
-L GND #PWR?
+L GND #PWR014
 U 1 1 59F848FA
 P 4600 6850
-F 0 "#PWR?" H 4600 6600 50  0001 C CNN
+F 0 "#PWR014" H 4600 6600 50  0001 C CNN
 F 1 "GND" H 4600 6700 50  0000 C CNN
 F 2 "" H 4600 6850 50  0001 C CNN
@@
 $EndComp
 $Comp
-L GND #PWR?
+L GND #PWR015
 U 1 1 59F84D94
 P 4700 6850
-F 0 "#PWR?" H 4700 6600 50  0001 C CNN
+F 0 "#PWR015" H 4700 6600 50  0001 C CNN
 F 1 "GND" H 4700 6700 50  0000 C CNN
 F 2 "" H 4700 6850 50  0001 C CNN
@@
 $EndComp
 $Comp
-L GND #PWR?
+L GND #PWR016
 U 1 1 59F8522E
 P 7550 11400
-F 0 "#PWR?" H 7550 11150 50  0001 C CNN
+F 0 "#PWR016" H 7550 11150 50  0001 C CNN
 F 1 "GND" H 7550 11250 50  0000 C CNN
 F 2 "" H 7550 11400 50  0001 C CNN
@@
 $EndComp
 $Comp
-L GND #PWR?
+L GND #PWR017
 U 1 1 59F8B68E
 P 9100 9550
-F 0 "#PWR?" H 9100 9300 50  0001 C CNN
+F 0 "#PWR017" H 9100 9300 50  0001 C CNN
 F 1 "GND" H 9100 9400 50  0000 C CNN
 F 2 "" H 9100 9550 50  0001 C CNN
@@
 $EndComp
 $Comp
-L GND #PWR?
+L GND #PWR018
 U 1 1 59F90123
 P 9800 10250
-F 0 "#PWR?" H 9800 10000 50  0001 C CNN
+F 0 "#PWR018" H 9800 10000 50  0001 C CNN
 F 1 "GND" H 9800 10100 50  0000 C CNN
 F 2 "" H 9800 10250 50  0001 C CNN
@@
 $EndComp
 $Comp
-L GND #PWR?
+L GND #PWR019
 U 1 1 59F93F86
 P 4450 12800
-F 0 "#PWR?" H 4450 12550 50  0001 C CNN
+F 0 "#PWR019" H 4450 12550 50  0001 C CNN
 F 1 "GND" H 4450 12650 50  0000 C CNN
 F 2 "" H 4450 12800 50  0001 C CNN
@@
 $EndComp
 $Comp
-L GND #PWR?
+L GND #PWR020
 U 1 1 59F9B00E
 P 8600 13000
-F 0 "#PWR?" H 8600 12750 50  0001 C CNN
+F 0 "#PWR020" H 8600 12750 50  0001 C CNN
 F 1 "GND" H 8600 12850 50  0000 C CNN
 F 2 "" H 8600 13000 50  0001 C CNN
@@
 $EndComp
 $Comp
-L GND #PWR?
+L GND #PWR021
 U 1 1 59FA0FDF
 P 27850 19150
-F 0 "#PWR?" H 27850 18900 50  0001 C CNN
+F 0 "#PWR021" H 27850 18900 50  0001 C CNN
 F 1 "GND" H 27850 19000 50  0000 C CNN
 F 2 "" H 27850 19150 50  0001 C CNN
@@
 $EndComp
 $Comp
-L GND #PWR?
+L GND #PWR022
 U 1 1 59FB3AF9
 P 5800 6400
-F 0 "#PWR?" H 5800 6150 50  0001 C CNN
+F 0 "#PWR022" H 5800 6150 50  0001 C CNN
 F 1 "GND" H 5800 6250 50  0000 C CNN
 F 2 "" H 5800 6400 50  0001 C CNN
@@
 	1    0    0    -1
 $EndComp
+Text Label 9700 13000 2    60   ~ 0
+LED3
+$Comp
+L LED LED7
+U 1 1 5A032909
+P 13950 4450
+F 0 "LED7" H 13950 4550 50  0000 C CNN
+F 1 "3mm" H 13950 4350 50  0000 C CNN
+F 2 "Keyboard:LED_D3.0mm" H 13950 4450 50  0001 C CNN
+F 3 "" H 13950 4450 50  0001 C CNN
+	1    13950 4450
+	1    0    0    -1
+$EndComp
+$Comp
+L LED LED8
+U 1 1 5A03FA67
+P 13950 4750
+F 0 "LED8" H 13950 4850 50  0000 C CNN
+F 1 "3mm" H 13950 4650 50  0000 C CNN
+F 2 "Keyboard:LED_D3.0mm" H 13950 4750 50  0001 C CNN
+F 3 "" H 13950 4750 50  0001 C CNN
+	1    13950 4750
+	1    0    0    -1
+$EndComp
+$Comp
+L R R9
+U 1 1 5A04A3A0
+P 14350 4450
+F 0 "R9" V 14430 4450 50  0000 C CNN
+F 1 "330R" V 14350 4450 50  0000 C CNN
+F 2 "Keyboard:R_0805" V 14280 4450 50  0001 C CNN
+F 3 "" H 14350 4450 50  0001 C CNN
+	1    14350 4450
+	0    -1   -1   0
+$EndComp
+$Comp
+L R R10
+U 1 1 5A051206
+P 14350 4750
+F 0 "R10" V 14430 4750 50  0000 C CNN
+F 1 "330R" V 14350 4750 50  0000 C CNN
+F 2 "Keyboard:R_0805" V 14280 4750 50  0001 C CNN
+F 3 "" H 14350 4750 50  0001 C CNN
+	1    14350 4750
+	0    -1   -1   0
+$EndComp
+Wire Wire Line
+	14200 4450 14100 4450
+Wire Wire Line
+	14100 4750 14200 4750
+Wire Wire Line
+	14500 4450 14550 4450
+Connection ~ 14550 4450
+Wire Wire Line
+	14500 4750 14550 4750
+Connection ~ 14550 4750
+Wire Wire Line
+	13600 4450 13800 4450
+Connection ~ 13600 3950
+Wire Wire Line
+	13600 4750 13800 4750
+Connection ~ 13600 4450
 $EndSCHEMATC
